Commit message: feat(phase-6): YOLO cleanup + TCP offset integration
- Remove all YOLO files, bboxes_ex_msgs package, and perception pipeline
- Clean CMakeLists.txt and package.xml of deleted dependencies
- Simplify reach.launch.py (robot + planner + control only)
- Add right_tcp_link to both URDF files (0.175m along wrist_yaw X)
- Planner default tip changed to right_tcp_link
- Add tcp_offset_x ROS parameter with KDL chain runtime override

File: src/unitree_g1_dex3_stack-main/robots/g1_description/g1_29dof_lock_waist_with_hand_rev_1_0.urdf (robot description, URDF)
Before this commit: robot g1_29dof_lock_waist_with_hand_rev_1_0, 54 links, 53 joints
Links:
- added link right_tcp_link
Joints:
- added joint right_tcp_joint: type fixed, parent right_wrist_yaw_link, child right_tcp_link, origin xyz=0.175 0 0 rpy=0 0 0

File: src/unitree_g1_dex3_stack-main/robots/g1_description/g1_29dof_lock_waist_with_hand_rev_1_0_collision_primitives.urdf (robot description, URDF)
Before this commit: robot g1_29dof_lock_waist_with_hand_rev_1_0, 54 links, 53 joints
Links:
- added link right_tcp_link
Joints:
- added joint right_tcp_joint: type fixed, parent right_wrist_yaw_link, child right_tcp_link, origin xyz=0.175 0 0 rpy=0 0 0
